Commit message: fix(issue-138): Clear servo-plate collision via mount offset
- Move Pendulum_Link servo mount: Y 0.0→6.5mm, Z 0.0→-15.0mm
  • Z shift clears all plates' local Z range [1.75, 7.25]
  • Y shift aligns servo shaft toward Base_Link edge (world-Z direction)
  • Verified collision cleared: servo Z-range [-31.81, -3.81] ≪ plates [-1.25, 1.25]

- Move Pendulum_Link_Right servo mount: Y 51.0→44.5mm, Z 6.0→-20.0mm
  • Z shift clears all plates' local Z range [-1.25, 4.25]
  • Y shift inverted (-6.5mm) due to roll=180° frame transform
  • Verified collision cleared: servo Z-range [-31.19, -3.19] ≪ plates [-1.25, 4.25]

Stage 7 (07_create_body_and_wheels.py) regenerated & verified.
Downstream stages (08-10) require live bridge to run; test suite passes.

Fixes #138

Co-Authored-By: Claude Haiku 4.5 <noreply@anthropic.com>
Claude-Session: https://claude.ai/code/session_016LAjYfZq92rw1E2657vRLY

File: inverted-pendulum-project/07_Simulation/webots/.generated/robot_webots.urdf (robot description, URDF)
Before this commit: robot inverted_pendulum_robot, 5 links, 4 joints
Links:
- link Pendulum_Link: geometry collision box size=0.032000 0.012000 0.028000; collision box size=0.059984 0.080033 0.005500
- link Pendulum_Link_Right: geometry collision box size=0.032000 0.012000 0.028000; collision box size=0.059984 0.080033 0.005500

Commit message: chore(#153): regenerate InvertedPendulumRobot.proto with updated Base_Link CoM
Reflects recent fix to Base_Link center of mass (Z: 0.089150 → 0.088650).
Also updates joint anchor positions and servo link translations.

Co-Authored-By: Claude Haiku 4.5 <noreply@anthropic.com>
Claude-Session: https://claude.ai/code/session_016LAjYfZq92rw1E2657vRLY

File: inverted-pendulum-project/07_Simulation/webots/.generated/robot_webots.urdf (robot description, URDF)
Before this commit: robot inverted_pendulum_robot, 5 links, 4 joints
Joints:
- joint wheel_left_joint: origin xyz=0.015001 -0.028526 0.054009 rpy=0.000000 0.000000 0.000000 -> xyz=0.014001 -0.028526 0.054010 rpy=0.000000 0.000000 0.000000
- joint wheel_right_joint: origin xyz=0.015001 0.067026 0.051009 rpy=0.000000 0.000000 0.000000 -> xyz=0.014001 0.073026 0.054010 rpy=0.000000 0.000000 0.000000
