Commit message: fix(issue-105): Add mesh scale attribute to servo visual geometry in URDF exporter
The servo visual mesh (feetech-STS3032-visual.stl) is authored in millimeters.
URDF expects coordinates in meters, so a scale attribute of [0.001, 0.001, 0.001]
must be present to convert mm to m. Without this, the mesh appears 1000x
oversized in simulators like Webots, causing physics explosion.

Changes:
- Add 'scale': [0.001, 0.001, 0.001] to Pendulum_Link servo mesh geometry dict
- Add 'scale': [0.001, 0.001, 0.001] to Pendulum_Link_Right servo mesh geometry dict
- Add test_servo_visual_mesh_has_scale() to verify scale attribute is present
  and correctly formatted in generated URDF

Fixes: #105

Co-Authored-By: Claude Haiku 4.5 <noreply@anthropic.com>
Claude-Session: https://claude.ai/code/session_016LAjYfZq92rw1E2657vRLY

File: inverted-pendulum-project/06_Exports/urdf/robot.urdf (robot description, URDF)
Before this commit: robot inverted_pendulum_robot, 5 links, 4 joints
Links:
- link Pendulum_Link: geometry collision box size=0.032000 0.012000 0.028000; collision box size=0.059984 0.005500 0.080033
- link Pendulum_Link_Right: geometry collision box size=0.032000 0.012000 0.028000; collision box size=0.059984 0.005500 0.080033

Commit message: fix(issue-121): Capture and export joint rotation in URDF
- 08_configure_assembly_joints.py: Extract rotation_ypr_deg from link Placement and save to joint_config.json
- 10_export_urdf.py: Add rpy parameter to build_urdf_joint(), convert joint rotation from degrees to radians (URDF format), and output in joint origin element
- test_urdf_fk_regression.py: Add test_joint_origin_rpy_matches_freecad_link_rotation() to verify joint rotations match FreeCAD metadata; remove KNOWN RISK #121 comment

Joint rotations now correctly captured:
- Wheel joints: identity [0, 0, 0] rad
- Pendulum_Link joint: roll=90° = [1.570796, 0, 0] rad (tilted so plates parallel wheel discs)
- Pendulum_Link_Right joint: roll=90° = [1.570796, 0, 0] rad

Fixes #121

Co-Authored-By: Claude Sonnet 5 <noreply@anthropic.com>
Claude-Session: https://claude.ai/code/session_016LAjYfZq92rw1E2657vRLY

File: inverted-pendulum-project/06_Exports/urdf/robot.urdf (robot description, URDF)
Before this commit: robot inverted_pendulum_robot, 5 links, 4 joints
Joints:
- joint pendulum_pivot_joint: origin xyz=-0.008001 -0.018276 0.070750 rpy=0 0 0 -> xyz=-0.008001 -0.018276 0.070750 rpy=1.570796 0.000000 0.000000
- joint pendulum_pivot_right_joint: origin xyz=-0.008001 0.062276 0.071250 rpy=0 0 0 -> xyz=-0.008001 0.062276 0.071250 rpy=1.570796 0.000000 0.000000
- joint wheel_left_joint: origin xyz=0.015001 -0.028526 0.054009 rpy=0 0 0 -> xyz=0.015001 -0.028526 0.054009 rpy=0.000000 0.000000 0.000000
- joint wheel_right_joint: origin xyz=0.015001 0.067026 0.054009 rpy=0 0 0 -> xyz=0.015001 0.067026 0.054009 rpy=0.000000 0.000000 0.000000

Commit message: fix(issue-143): Regenerate phase 8-10 artifacts with updated plate Z polarity
Phase 8 (Assembly Joint Configuration) now runs via FreeCAD MCP bridge with
correct Z-polarity values from phase 7:
- wheel_right_joint: Z=51.01mm (was stale 54.01mm)
- pendulum_pivot_right_joint: Z=68.25mm (was stale 71.25mm)

Propagated through phases 9-10:
- joint_config.json: fresh Z values in joint origins
- 09_mass_properties.json: computed from robot_assembly.FCStd
- 10_urdf_export_metadata.json: updated metadata
- robot.urdf: Z-corrected joint positions
- robot_webots.urdf: regenerated for Webots integration
- InvertedPendulumRobot.proto: Webots PROTO with corrected joint geometry

All 3 previously failing Z-polarity tests now pass:
✓ test_wheel_right_joint_origin_matches_link_placement
✓ test_pendulum_pivot_right_joint_origin_matches_link_placement
✓ test_joint_origin_transitively_matches_freecad_link_placement

Full test suite: 200 passed, 1 skipped (issue-143, issue-135)

Co-Authored-By: Claude Haiku 4.5 <noreply@anthropic.com>
Claude-Session: https://claude.ai/code/session_016LAjYfZq92rw1E2657vRLY

File: inverted-pendulum-project/06_Exports/urdf/robot.urdf (robot description, URDF)
Before this commit: robot inverted_pendulum_robot, 5 links, 4 joints
Joints:
- joint pendulum_pivot_right_joint: origin xyz=-0.008001 0.062276 0.071250 rpy=1.570796 0.000000 0.000000 -> xyz=-0.008001 0.062276 0.068250 rpy=1.570796 0.000000 0.000000
- joint wheel_right_joint: origin xyz=0.015001 0.067026 0.054009 rpy=0.000000 0.000000 0.000000 -> xyz=0.015001 0.067026 0.051009 rpy=0.000000 0.000000 0.000000

File: inverted-pendulum-project/07_Simulation/webots/.generated/robot_webots.urdf (robot description, URDF)
Before this commit: robot inverted_pendulum_robot, 5 links, 4 joints
Links:
- link Pendulum_Link: geometry collision box size=0.032000 0.012000 0.028000; collision box size=0.059984 0.080033 0.005500
- link Pendulum_Link_Right: geometry collision box size=0.032000 0.012000 0.028000; collision box size=0.059984 0.080033 0.005500
Joints:
- joint pendulum_pivot_right_joint: origin xyz=-0.008001 0.062276 0.071250 rpy=1.570796 0.000000 0.000000 -> xyz=-0.008001 0.062276 0.068250 rpy=1.570796 0.000000 0.000000
- joint wheel_right_joint: origin xyz=0.015001 0.067026 0.054009 rpy=0.000000 0.000000 0.000000 -> xyz=0.015001 0.067026 0.051009 rpy=0.000000 0.000000 0.000000

Commit message: chore(issue-146): regenerate phases 7-10 on rebased #144 baseline
After rebasing onto merged #144 (which restored the #143 plate-Z-
polarity fix and #138 servo-position fix), regenerate all downstream
artifacts so they reflect the full 6-entry placement_overrides.yaml
applied on top of the now-correct baseline constants.

Confirms the container-Z asymmetry reported during visual review is
gone: Wheel_Left/Wheel_Right now share the exact same Z (53.5095mm,
range [38.51,68.51] both sides) -- previously [38.51,68.51] vs
[41.51,71.51], a 0.5mm-to-3mm compounding asymmetry traced (Architect
investigation) to the pre-#144 stale PENDULUM_LINK_RIGHT_TOP_PLATE_Z_MM/
_MIDDLE_PLATE_Z_MM constants, unrelated to the override mechanism
itself.

Full suite: 221 passed, 0 skipped, 0 failed (up from 216 passed / 5
failed pre-regen -- those 5 were exactly this stale-artifact mismatch,
not defects in #146's mechanism).

Co-Authored-By: Claude Sonnet 5 <noreply@anthropic.com>
Claude-Session: https://claude.ai/code/session_016LAjYfZq92rw1E2657vRLY

File: inverted-pendulum-project/06_Exports/urdf/robot.urdf (robot description, URDF)
Before this commit: robot inverted_pendulum_robot, 5 links, 4 joints
Joints:
- joint wheel_left_joint: origin xyz=0.015001 -0.028526 0.054009 rpy=0.000000 0.000000 0.000000 -> xyz=0.014001 -0.028526 0.053509 rpy=0.000000 0.000000 0.000000
- joint wheel_right_joint: origin xyz=0.015001 0.067026 0.051009 rpy=0.000000 0.000000 0.000000 -> xyz=0.014001 0.073026 0.053509 rpy=0.000000 0.000000 0.000000

Commit message: feat(issue-146): implement split-axis wheel Z correction for Amendment 2
Implementation of Issue #146 Amendment 2: wheel placement handling now uses
split-axis logic:
  - X/Y axes: remain verify-only (hole-derived, physical hole-fit invariant)
  - Z axis: now APPLIED from YAML adjust[2] if it differs beyond tolerance

Changes:
1. Modified _verify_wheel_expected_position() to compare X/Y against YAML
   (warn-only) and apply Z correction when needed, printing distinct
   confirmation messages for each axis.

2. Updated test_placement_overrides.py to verify split-axis behavior:
   - X/Y remain hole-derived (don't match YAML targets)
   - Z is applied (must match YAML adjust[2])
   - Added test_wheel_split_axis_z_applied_xy_hole_derived() to verify behavior
   - Updated test_wheel_split_axis_mechanism_runs() to check for Z messages

3. Updated placement_overrides.yaml comment to reflect split-axis semantics

4. Regenerated full pipeline:
   Phase 7: Wheel Z now corrected to 54.01mm (per YAML)
   Phase 8: Joint origins reflect corrected wheel positions
   Phase 9: Mass properties computed with correct wheel positions
   Phase 10: URDF generated with wheel joints at Z=0.054010m

Wheel positions after regen:
  Wheel_Left: (14.0007, -28.5258, 54.01) mm
  Wheel_Right: (14.0007, 73.0258, 54.01) mm
  Both Z values now match YAML adjust[2]=54.01, X/Y remain hole-derived.

Fixes #146
Co-Authored-By: Claude Haiku 4.5 <noreply@anthropic.com>
Claude-Session: https://claude.ai/code/session_016LAjYfZq92rw1E2657vRLY

File: inverted-pendulum-project/06_Exports/urdf/robot.urdf (robot description, URDF)
Before this commit: robot inverted_pendulum_robot, 5 links, 4 joints
Joints:
- joint wheel_left_joint: origin xyz=0.014001 -0.028526 0.053509 rpy=0.000000 0.000000 0.000000 -> xyz=0.014001 -0.028526 0.054010 rpy=0.000000 0.000000 0.000000
- joint wheel_right_joint: origin xyz=0.014001 0.073026 0.053509 rpy=0.000000 0.000000 0.000000 -> xyz=0.014001 0.073026 0.054010 rpy=0.000000 0.000000 0.000000

Commit message: fix(#156): regenerate robot.urdf with correct pendulum pivot axes, enhance validator with direction check
- Regenerate robot.urdf with corrected pendulum_pivot_joint and pendulum_pivot_right_joint axes
  from [0,1,0] (incorrect) to [0,0,-1] (correct). Axes are now properly composed from global
  axis with inverse RPY rotation matrix.

  For pendulum pivots with rpy=[0,0,π/2] (90° roll about X):
  - Global axis [0,1,0] is rotated to [0,0,-1] in the child frame (issue #156).
  - Wheel joints maintain [0,1,0] as expected (no RPY rotation applied).

- Enhance validate_joint_axes() in 12_validate_urdf_export.py with axis direction validation:
  - Add ypr_deg_to_rotation_matrix() helper for axis composition
  - Add compose_axis() to compute expected axis from global axis + RPY rotation
  - Add load_joint_config() to load joint metadata
  - Update validate_joint_axes() to check both unit vector norm AND axis direction
  - Direction check verifies URDF axis matches expected composed value (tolerance 1e-3)
  - Previous validator only checked norm ≈ 1.0, which could not detect direction errors

- Update all downstream generated artifacts (metadata, validation reports)

All tests pass (36/36):
  - test_joint_axes passes with correct [0,0,-1] axis values
  - test_urdf_fk_regression passes
  - Validator passes all 4 checks including new direction validation

Co-Authored-By: Claude Haiku 4.5 <noreply@anthropic.com>
Claude-Session: https://claude.ai/code/session_016LAjYfZq92rw1E2657vRLY

File: inverted-pendulum-project/06_Exports/urdf/robot.urdf (robot description, URDF)
Before this commit: robot inverted_pendulum_robot, 5 links, 4 joints
Joints:
- joint pendulum_pivot_joint: axis 0.000000 1.000000 0.000000 -> 0.000000 0.000000 -1.000000
- joint pendulum_pivot_right_joint: axis 0.000000 1.000000 0.000000 -> 0.000000 0.000000 -1.000000
